Commit message: modified control launch file, add yaml for controller and change cmake

File: ros2_control/quad_bot.xacro (robot description, xacro)
@@ -4,6 +4,6 @@
   <xacro:include filename="$(find quad_bot_description)/urdf/quad_bot.xacro"/>
   <!-- create link fixed to the "world" -->
-  <link name="world"/>
-  <xacro:quad_bot/>
+  <!-- <link name="world"/>
+  <xacro:quad_bot/> -->
   <!-- Import quad ros2_control description -->
   <xacro:include filename="$(find quad_bot_controller)/ros2_control/quad.ros2_control.xacro" />

Commit message: add change to xacro

File: ros2_control/quad_bot.xacro (robot description, xacro)
@@ -4,6 +4,13 @@
   <xacro:include filename="$(find quad_bot_description)/urdf/quad_bot.xacro"/>
   <!-- create link fixed to the "world" -->
-  <!-- <link name="world"/>
-  <xacro:quad_bot/> -->
+  <link name="world"/>
+<!--
+  <joint name="base_joint" type="fixed">
+    <parent link="world"/>
+    <child link="base_link"/>
+    <origin xyz="0 0 0" rpy="0 0 0"/>
+    <axis xyz="0 0 1"/>
+  </joint> -->
+  <!-- <xacro:quad_bot/> -->
   <!-- Import quad ros2_control description -->
   <xacro:include filename="$(find quad_bot_controller)/ros2_control/quad.ros2_control.xacro" />
